File: stm32_canbus_module.kicad_pcb (KiCad board)
At the start: 2 copper layers, 33 x 33 mm, 20 parts, among them J11 Conn_01x10, J5 Conn_01x10, J6 Conn_01x10, J7 Conn_01x10, U1 STM32L431CCTx, U2 TLE9251, U3 AP7384-28Y, X1 ASE-8.000MHZ-LC-T

Commit message: v1.1
Parts:
- added C2: 100nF, Capacitor_SMD:C_0603_1608Metric_Pad1.08x0.95mm_HandSolder, F.Cu at (155.3, 106.4)
- U3: value AP7384-28Y -> AP7384-33Y
- moved C5 0.65 mm to (156.0, 101.8)
Connections:
- C8 pad 1: VIN -> 5V
- J11 pad 10: VIN -> 5V
- U2 pad 3: 3V3 -> 5V
- U3 pad 3: VIN -> 5V
Routing:
- net 5V: track 0.00 -> 40.0 mm, vias 0 -> 2
- net VIN: track 6.73 -> 0.00 mm
- net 3V3: track 92.2 -> 89.4 mm, vias 0 -> 1
Other:
- board text added: "1.1 CAN transceiver connected to VIN instead of 3.3V"
- board text added: "stm32-canbus-module v1.1 - 2023/03/01 Cedric Priscal"
- board text removed: "stm32-canbus-module v1.0 - 2022/12/01 Cedric Priscal"
