File: stm32_canbus_module.kicad_sch (KiCad schematic)
At the start: 20 parts, among them J11 Conn_01x10, J5 Conn_01x10, J6 Conn_01x10, J7 Conn_01x10, U1 STM32L431CCTx, U2 TLE9251, U3 AP7384-28Y, X1 ASE-8.000MHZ-LC-T

Commit message: Updating BOM
Parts:
- C1: DigiKey (none) -> 490-4781-1-ND
- C10, C11, C4, C5, C6, C7: DigiKey (none) -> 1276-1000-1-ND
- C12: DigiKey (none) -> 1276-2910-1-ND
- C3: DigiKey (none) -> 1276-1244-1-ND
- C8, C9: DigiKey (none) -> 587-2229-1-ND
- R1: DigiKey (none) -> RNCP0603FTD10K0CT-ND
- U3: value AP7384-28Y -> AP7384-33Y; DigiKey (none) -> AP7384-33Y-13DICT-ND
Other:
- moved on the sheet: C1, C10, C3, C4, C6, C7, C8, C9, U3

Commit message: v1.1
Parts:
- added C2: 100nF, Capacitor_SMD:C_0603_1608Metric_Pad1.08x0.95mm_HandSolder, symbol Device:C
Connections:
- net 3V3: no longer U2.3 (VCC)
- net GND: now also C2.2
- net VIN renamed 5V
- net 5V: now also U2.3 (VCC), C2.1
Other:
- note added: "Add 5V regulator?"
- moved on the sheet: C11, C12
