File: stm32_canbus_module.kicad_sch (KiCad schematic)
At the start: 21 parts, among them J11 Conn_01x10, J5 Conn_01x10, J6 Conn_01x10, J7 Conn_01x10, U1 STM32L431CCTx, U2 TLE9251, U3 AP7384-33Y, X1 ASE-8.000MHZ-LC-T

Commit message: 2.0
- Adding 5V regulator, VIN now supports 12V
- Migration to KiCad 9
Parts:
- removed C12: 22uF, Capacitor_SMD:C_0805_2012Metric_Pad1.18x1.45mm_HandSolder, symbol Device:C
- removed C3: 4.7uF, Capacitor_SMD:C_0805_2012Metric_Pad1.18x1.45mm_HandSolder, symbol Device:C
- added C10: 10uF, Capacitor_SMD:C_0805_2012Metric_Pad1.18x1.45mm_HandSolder, symbol Device:C
- added U2: AP7384-33Y, Package_TO_SOT_SMD:SOT-89-3, symbol Regulator_Linear:AP7384-28Y
- C11: renamed from C9; value 1uF -> 10uF; DigiKey 587-2229-1-ND -> 399-C0805C106K8PACTUCT-ND
- C8: value 1uF -> 2.2uF; footprint Capacitor_SMD:C_0805_2012Metric_Pad1.18x1.45mm_HandSolder -> Capacitor_SMD:C_0603_1608Metric_Pad1.08x0.95mm_HandSolder; DigiKey 587-2229-1-ND -> 490-10731-1-ND
- renumbered C5 to C1, C11 to C12, C2 to C14, C1 to C2, C6 to C4, C4 to C5, C7 to C6, C10 to C7, J6 to J1, J7 to J2, J5 to J3, J11 to J4, U2 to U4
Connections:
- net 5V: now also C10.1, U2.1 (VO); no longer C8.1, J4.10 (Pin_10), U3.3 (VI)
- net GND: now also C10.2, U2.2 (GND)
- new net VIN: C8.1, J4.10 (Pin_10), U2.3 (VI), U3.3 (VI)
Other:
- note added: "TODO replace by AP7375"
- note removed: "Add 5V regulator?"
- moved on the sheet: C11, U3
